File: hardware/coin1.kicad_pcb (KiCad board)
At the start: 2 copper layers, 140 x 40 mm, 73 parts, among them J1 Conn_01x04, J2 Conn_01x03, T1 TestPoint_THTPad_3.0x3.0mm_Dr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, T10 TestPoint_THTPad_3.0x3.0mm_Dr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, T11 TestPoint_THTPad_3.0x3.0mm_Dr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, T12 TestPoint_THTPad_3.0x3.0mm_Dr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, T2 TestPoint_THTPad_3.0x3.0mm_Dr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, T22 TestPoint_THTPad_D1.0mm_Drill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, T23 TestPoint_THTPad_D1.0mm_Drill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, T24 TestPoint_THTPad_D1.0mm_Drill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

Commit message: add locations for JLCPCB order IDs
Other:
- board text added: "JLCJLCJLCJLC"
Changed lines of the file:
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@@
 		)
 		(fp_text user "${REFERENCE}"
-			(at 0 -3.81 360)
+			(at 0 -3.81 0)
 			(layer "B.Fab")
 			(effects
@@
 			)
 		)
+	)
+	(gr_rect
+		(start 145 42)
+		(end 155 52)
+		(stroke
+			(width 0.1)
+			(type solid)
+		)
+		(fill solid)
+		(layer "F.SilkS")
 	)
 	(gr_poly
@@
 		(layer "User.2")
 	)
+	(gr_text "JLCJLCJLCJLC"
+		(at 107 47 0)
+		(layer "F.SilkS")
+		(effects
+			(font
+				(size 1 1)
+				(thickness 0.1)
+			)
+			(justify left bottom)
+		)
+	)
+	(gr_text "JLCJLCJLCJLC"
+		(at 57 47 0)
+		(layer "F.SilkS")
+		(effects
+			(font
+				(size 1 1)
+				(thickness 0.1)
+			)
+			(justify left bottom)
+		)
+	)
 	(segment

Commit message: add LCSC part details
Parts:
- R1, R10, R2, R3, R4, R5, R6, R7, R8, R9: value R -> 47R
Connections:
- U1 pad 21: GND -> VSS
