File: hardware/b4/b4.kicad_pcb (KiCad board)
At the start: 2 copper layers, 40 x 40 mm, 13 parts, among them T42 TestPoint_THTPad_D1.0mm_Drill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, T43 TestPoint_THTPad_D1.0mm_Drill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, T44 TestPoint_THTPad_D1.0mm_Drill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, T45 TestPoint_THTPad_D1.0mm_Drill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, T46 TestPoint_THTPad_D1.0mm_Drill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, T48 TestPoint_THTPad_D1.0mm_Drill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, T49 TestPoint_THTPad_D1.0mm_Drill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, T50 TestPoint_THTPad_D1.0mm_Drill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, T51 TestPoint_THTPad_D1.0mm_Drill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, T52 TestPoint_THTPad_D1.0mm_Drill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

Commit message: update fab output
Other:
- board text added: "LIMITED EDITION"
Changed lines of the file:
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@@
 			(drillshape 0)
 			(scaleselection 1)
-			(outputdirectory "")
+			(outputdirectory "fab/")
 		)
 	)
@@
 	)
 	(gr_rect
-		(start 145 42)
-		(end 155 52)
+		(start 145 32)
+		(end 155 42)
 		(stroke
 			(width 0.1)
@@
 		(fill solid)
 		(layer "F.SilkS")
+	)
+	(gr_rect
+		(start 132.6 48.3)
+		(end 167.4 51.4)
+		(stroke
+			(width 1)
+			(type solid)
+		)
+		(fill solid)
+		(layer "F.Mask")
 	)
 	(gr_circle
@@
 		(layer "User.2")
 	)
+	(gr_text "LIMITED EDITION"
+		(at 150 50 0)
+		(layer "F.Cu")
+		(effects
+			(font
+				(size 3 3)
+				(thickness 0.5)
+				(bold yes)
+			)
+		)
+	)
 	(segment
