File: hardware/SAO-CR1616/SAO-CR1616.kicad_pcb (KiCad board)
At the start: 2 copper layers, 16 x 29.5 mm, 5 parts, among them J2 SAO v1.69bis addon

Commit message: separate into fab-able parts
Parts:
- added ?: , , F.Cu at (65.1, 152.8)
- added ?: , , F.Cu at (65.1, 149.8)
- added ?: , , F.Cu at (62.9, 149.2)
- added ?: , , F.Cu at (62.9, 153.2)
- added ?: , , F.Cu at (65.1, 151.8)
- added ?: , , F.Cu at (62.9, 150.2)
- added ?: , , F.Cu at (65.1, 150.8)
- added ?: , , F.Cu at (65.1, 151.3)
- added ?: , , F.Cu at (62.9, 151.7)
- added ?: , , F.Cu at (62.9, 149.7)
- added ?: , , F.Cu at (62.9, 152.7)
- added ?: , , F.Cu at (65.1, 150.3)
- added ?: , , F.Cu at (62.9, 148.7)
- added ?: , , F.Cu at (65.1, 148.8)
- added ?: , , F.Cu at (62.9, 151.2)
- added ?: , , F.Cu at (62.9, 152.2)
- added ?: , , F.Cu at (62.9, 150.7)
- added ?: , , F.Cu at (65.1, 153.3)
- added ?: , , F.Cu at (65.1, 152.3)
- added ?: , , F.Cu at (65.1, 149.3)
- added BC1: 1u, Capacitor_SMD:C_0805_2012Metric_Pad1.18x1.45mm_HandSolder, B.Cu at (40.7, 146.0)
- added BC2: 1u, Capacitor_SMD:C_0805_2012Metric_Pad1.18x1.45mm_HandSolder, B.Cu at (50.0, 146.0)
- added BC3: 1u, Capacitor_SMD:C_0805_2012Metric_Pad1.18x1.45mm_HandSolder, B.Cu at (59.3, 146.0)
- added BC4: 1u, Capacitor_SMD:C_0805_2012Metric_Pad1.18x1.45mm_HandSolder, B.Cu at (59.3, 154.0)
- added BC5: 1u, Capacitor_SMD:C_0805_2012Metric_Pad1.18x1.45mm_HandSolder, B.Cu at (50.0, 154.0)
- added BC6: 1u, Capacitor_SMD:C_0805_2012Metric_Pad1.18x1.45mm_HandSolder, B.Cu at (40.7, 154.0)
- added BC7: 1u, Capacitor_SMD:C_0805_2012Metric_Pad1.18x1.45mm_HandSolder, B.Cu at (45.3, 150.0)
- added J3: SAO v1.69bis badge, Connector_IDC:IDC-Header_2x03_P2.54mm_Vertical, F.Cu at (52.5, 148.7)
- added P1: Conn_01x02, Connector_PinHeader_2.54mm:PinHeader_1x02_P2.54mm_Vertical, B.Cu at (41.9, 142.0)
- added P2: Conn_01x02, Connector_PinHeader_2.54mm:PinHeader_1x02_P2.54mm_Vertical, B.Cu at (51.3, 142.0)
- added P3: Conn_01x02, Connector_PinHeader_2.54mm:PinHeader_1x02_P2.54mm_Vertical, B.Cu at (60.6, 142.0)
- added P4: Conn_01x02, Connector_PinHeader_2.54mm:PinHeader_1x02_P2.54mm_Vertical, B.Cu at (58.1, 158.0)
- added P5: Conn_01x02, Connector_PinHeader_2.54mm:PinHeader_1x02_P2.54mm_Vertical, B.Cu at (48.7, 158.0)
- added P6: Conn_01x02, Connector_PinHeader_2.54mm:PinHeader_1x02_P2.54mm_Vertical, B.Cu at (39.4, 158.0)
- moved B3 77.6 mm to (73.0, 140.3)
- moved B4 77.6 mm to (73.0, 140.3)
- moved SAO-P1 77.6 mm to (73.0, 140.3)
- moved SAO-P2 77.6 mm to (73.0, 140.3)
- moved J2 77.6 mm to (70.5, 155.4)
Routing:
- net +3V0: track 16.2 -> 43.1 mm
- net GND: track 22.5 -> 49.3 mm
- added copper zone on F.Cu, net +3V0
Other:
- board size 16 x 29.5 mm -> 44 x 29.7 mm
- board text added: "JLCJLCJLCJLC"
