File: hardware/smd0402/smd0402.kicad_pcb (KiCad board)
At the start: 2 copper layers, 150 x 146.5 mm, 124 parts, among them J1 Conn_01x03, J2 SAO v1.69bis addon, U1 WCH CH32V003F4U6

Commit message: tweak instructions
Other:
- board text added: "to align use 1.0mm dia pins"
Changed lines of the file:
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@@
+	)
+	(gr_line
+		(start 61.16 50.13)
+		(end 72.26 47.28)
+		(stroke
+			(width 0.1)
+			(type default)
+		)
+		(layer "F.SilkS")
+	)
+	(gr_line
+		(start 38.86 50.19)
+		(end 27.82 47.28)
+		(stroke
+			(width 0.1)
+			(type default)
+		)
+		(layer "F.SilkS")
+	)
+	(gr_line
+		(start 61.16 50.13)
+		(end 72.21 52.44)
+		(stroke
+			(width 0.1)
+			(type default)
+		)
+		(layer "F.SilkS")
 	)
 	(gr_line
@@
 			(xy 42.06 39.34) (xy 43.57 60.75) (xy 55.49 44.02) (xy 72.822 55.156)
 		)
+		(stroke
+			(width 0.1)
+			(type default)
+		)
+		(layer "F.SilkS")
+	)
+	(gr_line
+		(start 38.86 50.19)
+		(end 27.8 52.41)
 		(stroke
 			(width 0.1)
@@
 		(layer "B.SilkS")
 	)
+	(gr_line
+		(start 138.25 50.08)
+		(end 127.74 47.27)
+		(stroke
+			(width 0.1)
+			(type default)
+		)
+		(layer "B.SilkS")
+	)
 	(gr_poly
 		(pts
@@
 	(gr_curve
 		(pts
-			(xy 153.095 39.346224) (xy 148.26 59.36) (xy 143.73 63.33) (xy 138.49 69.82)
+			(xy 153.095 39.346224) (xy 151.04 59.39) (xy 143.73 63.33) (xy 138.49 69.82)
 		)
 		(stroke
@@
 		(layer "B.SilkS")
 	)
+	(gr_line
+		(start 161.22 50.08)
+		(end 172.2 47.23)
+		(stroke
+			(width 0.1)
+			(type default)
+		)
+		(layer "B.SilkS")
+	)
 	(gr_poly
 		(pts
@@
 		(layer "B.SilkS")
 	)
+	(gr_line
+		(start 138.25 50.08)
+		(end 127.71 52.49)
+		(stroke
+			(width 0.1)
+			(type default)
+		)
+		(layer "B.SilkS")
+	)
 	(gr_poly
 		(pts
@@
 		(fill yes)
 		(locked yes)
+		(layer "B.SilkS")
+	)
+	(gr_line
+		(start 161.22 50.08)
+		(end 172.14 52.4)
+		(stroke
+			(width 0.1)
+			(type default)
+		)
 		(layer "B.SilkS")
 	)
@@
 		)
 	)
+	(gr_text "to align use 1.0mm dia pins"
+		(at 50 50 0)
+		(layer "F.SilkS")
+		(effects
+			(font
+				(size 1 1)
+				(thickness 0.1)
+			)
+		)
+	)
 	(gr_text "3. apply solder paste,\n   reflow to thicken pad"
 		(at 52.68 61.62 0)
@@
 	(gr_text "JLCJLCJLCJLC"
 		(locked yes)
-		(at 60 50 0)
+		(at 62 47 0)
 		(layer "F.SilkS")
 		(effects
@@
 		)
 	)
+	(gr_text "to align use 1.0mm dia pins"
+		(at 150 50 0)
+		(layer "B.SilkS")
+		(effects
+			(font
+				(size 1 1)
+				(thickness 0.1)
+			)
+			(justify mirror)
+		)
+	)
