File: hardware/reverse-panel/reverse-panel-cleaned.kicad_pcb (KiCad board)
At the start: 2 copper layers, 116 x 102 mm, 120 parts

Commit message: update rails+mousebites empty panel
Other:
- board text added: "jlcpcb.com/help/article/How-to-remove-order-number-from-your-PCB jlcpcb.com/help/article/Panelizing-your-PCB-for-Assembly jlcpcb.com/help/article/How-to-add-tooling-holes-for-PCB-assembly-order"
Changed lines of the file:
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@@
 		(layer "User.2")
+	)
+	(gr_text "jlcpcb.com/help/article/How-to-remove-order-number-from-your-PCB\njlcpcb.com/help/article/Panelizing-your-PCB-for-Assembly\njlcpcb.com/help/article/How-to-add-tooling-holes-for-PCB-assembly-order\n"
+		(at 131.05 130.01 0)
+		(layer "Cmts.User")
+		(effects
+			(font
+				(size 1 1)
+				(thickness 0.15)
+			)
+			(justify left top)
+		)
 	)
 	(zone
