File: hardware/reverse/reverse.kicad_pcb (KiCad board)
At the start: 2 copper layers, 50 x 50 mm, 52 parts, among them J1 Conn_01x03, U1 WCH CH32V003F4U6

Commit message: cleanup fab files
Parts:
- added align-r1: , , F.Cu at (27.8, 47.3)
- added align-r4: , , F.Cu at (72.2, 52.4)
- moved R2 8.36 mm to (32.4, 58.4)
- moved R7 8.36 mm to (67.6, 58.4)
- renumbered align-r1 to align-r3
Routing:
- net GND: track 4.28 -> 19.0 mm, vias 119 -> 106
- net /touch2: track 8.69 -> 16.7 mm
- net GP7: track 38.6 -> 34.8 mm
- net PWM2: track 16.3 -> 19.8 mm
- net PWM7: track 16.5 -> 20.0 mm
- net GP2: track 38.3 -> 35.1 mm
- net /touch1: track 17.2 -> 17.9 mm, vias 1 -> 3
Other:
- board text removed: "import QR SVG scale 0.2"

Commit message: separate boards
Parts:
- removed through-r1, through-r2, through-r3, through-r4, through-r5, through-r6, through-r7: TestPoint_THTPad_D2.0mm_Drill1.0mm, TestPoint:TestPoint_THTPad_D2.0mm_Drill1.0mm
- added contact-r1: TestPoint_Pad_D4.0mm, TestPoint:TestPoint_Pad_D4.0mm, F.Cu at (45.0, 42.2)
- stitch1 (x11): value (none) -> TestPoint_Pad_D2.0mm; footprint (none) -> TestPoint:TestPoint_Pad_D2.0mm
Routing:
- net GND: vias 106 -> 105
- net +3V0: vias 14 -> 21
Other:
- board text added: "3. apply solder paste, reflow to thicken pad"
- board text added: "4. apply solder paste, stack upper sandwich, reflow"
- board text added: "to align use 1.0mm dia pins"
- board text removed: "github.com/eutectic6337/coin1"
