File: hardware/reverse/reverse.kicad_pcb (KiCad board)
At the start: 2 copper layers, 50 x 50 mm, 48 parts, among them J1 Conn_01x03, U1 CH32V003F4U6

Commit message: latest separated fabricated boards
Routing:
- net GND: vias 105 -> 116
Changed lines of the file:
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@@
+	)
+	(via
+		(at 53 68)
+		(size 0.5)
+		(drill 0.3)
+		(layers "F.Cu" "B.Cu")
+		(free yes)
+		(net 2)
 	)
 	(via
@@
 	)
 	(via
+		(at 51 66.5)
+		(size 0.5)
+		(drill 0.3)
+		(layers "F.Cu" "B.Cu")
+		(free yes)
+		(net 2)
+	)
+	(via
 		(at 43.434 45.8)
 		(size 0.5)
@@
 	)
 	(via
+		(at 50 69)
+		(size 0.5)
+		(drill 0.3)
+		(layers "F.Cu" "B.Cu")
+		(free yes)
+		(net 2)
+	)
+	(via
 		(at 66.802 34.1)
 		(size 0.6)
@@
 	)
 	(via
+		(at 50 60)
+		(size 0.5)
+		(drill 0.3)
+		(layers "F.Cu" "B.Cu")
+		(free yes)
+		(net 2)
+	)
+	(via
 		(at 41.659829 36.176508)
 		(size 0.6)
@@
 	)
 	(via
+		(at 47.5 62)
+		(size 0.5)
+		(drill 0.3)
+		(layers "F.Cu" "B.Cu")
+		(free yes)
+		(net 2)
+	)
+	(via
 		(at 54.590219 42.30831)
 		(size 0.6)
@@
 	)
 	(via
+		(at 53 61)
+		(size 0.5)
+		(drill 0.3)
+		(layers "F.Cu" "B.Cu")
+		(free yes)
+		(net 2)
+	)
+	(via
 		(at 43.712243 64.070243)
 		(size 0.5)
@@
 	)
 	(via
+		(at 50 64.5)
+		(size 0.5)
+		(drill 0.3)
+		(layers "F.Cu" "B.Cu")
+		(free yes)
+		(net 2)
+	)
+	(via
 		(at 55.294048 27.322727)
 		(size 0.6)
@@
 	)
 	(via
+		(at 45.5 64.5)
+		(size 0.5)
+		(drill 0.3)
+		(layers "F.Cu" "B.Cu")
+		(free yes)
+		(net 2)
+	)
+	(via
 		(at 52.578 53.378)
 		(size 0.5)
@@
 	)
 	(via
+		(at 54.5 64.5)
+		(size 0.5)
+		(drill 0.3)
+		(layers "F.Cu" "B.Cu")
+		(free yes)
+		(net 2)
+	)
+	(via
 		(at 29.2 42.825258)
 		(size 0.6)
@@
 	)
 	(via
+		(at 47.5 67)
+		(size 0.5)
+		(drill 0.3)
+		(layers "F.Cu" "B.Cu")
+		(free yes)
+		(net 2)
+	)
+	(via
 		(at 39.37 34.794)
 		(size 0.5)
@@
 		(drill 0.3)
 		(layers "F.Cu" "B.Cu")
+		(free yes)
+		(net 2)
+	)
+	(via
+		(at 51 62.5)
+		(size 0.5)
+		(drill 0.3)
+		(layers "F.Cu" "B.Cu")

Commit message: prep for another fab run
Parts:
- added solder1: TestPoint_Pad_D1.0mm, TestPoint:TestPoint_Pad_D1.0mm, B.Cu at (44.9, 42.2)
- added solder2: TestPoint_Pad_D1.0mm, TestPoint:TestPoint_Pad_D1.0mm, B.Cu at (44.9, 41.5)
- added solder3: TestPoint_Pad_D1.0mm, TestPoint:TestPoint_Pad_D1.0mm, B.Cu at (45.5, 41.8)
- added solder4: TestPoint_Pad_D1.0mm, TestPoint:TestPoint_Pad_D1.0mm, B.Cu at (45.5, 42.6)
- added solder5: TestPoint_Pad_D1.0mm, TestPoint:TestPoint_Pad_D1.0mm, B.Cu at (44.9, 42.9)
- added solder6: TestPoint_Pad_D1.0mm, TestPoint:TestPoint_Pad_D1.0mm, B.Cu at (44.3, 42.6)
- added solder7: TestPoint_Pad_D1.0mm, TestPoint:TestPoint_Pad_D1.0mm, B.Cu at (44.3, 41.8)
- moved battery-eject1 2.00 mm to (50.0, 59.0)
Routing:
- net GND: vias 116 -> 125
- net +3V0: vias 21 -> 14
Other:
- board text added: "import QR SVG scale 0.2"
- board text added: "import rear (Inkscape) SVG scale 0.075"

Commit message: update fab files
Other:
- board text removed: "import QR SVG scale 0.2"
- board text removed: "import rear (Inkscape) SVG scale 0.075"
